File: hardware/Gateometry.kicad_sch (KiCad schematic)
At the start: 66 parts, among them J1 POWER, J10 CLOCK OUT, J2 GATE1, J3 GATE3, J4 GATE5, J5 GATE7, J6 GATE2, J7 GATE4, J8 GATE6, J9 GATE8, SW1 RUN/STOP, SW2 MUTE 1, SW3 MUTE 2, SW4 MUTE 3, SW5 MUTE 4, SW6 MUTE 5, SW7 MUTE 6, SW8 MUTE 7, SW9 MUTE 8, U1 74HC595, U2 74HC165, U4 74HCT541, U5 74HCT541

Commit message: initial final rev A schematic
Parts:
- added C5, C6, C7: 100n, Capacitor_THT:C_Disc_D3.0mm_W1.6mm_P2.50mm, symbol Device:C
- added D11, D12: BAT85, Diode_THT:D_DO-35_SOD27_P7.62mm_Horizontal, symbol Diode:BAT85
- added J10: CLOCK IN, Desval27:Jack_3.5mm_QingPu_WQP-PJ398SM_Vertical, symbol Desval27:3.5mm_Mono_Switched_Jack
- added R23: 22k, Resistor_THT:R_Axial_DIN0207_L6.3mm_D2.5mm_P2.54mm_Vertical, symbol Device:R
- added R24: 100k, Resistor_THT:R_Axial_DIN0207_L6.3mm_D2.5mm_P2.54mm_Vertical, symbol Device:R
- added U5: 74HCT14, Package_DIP:DIP-14_W7.62mm_LongPads, symbol 74xx:74HC14
- C1: renamed from C2; value 10µF -> 47µ
- R1: renamed from R5; value 1kΩ -> 1k
- R10: renamed from R4; value 10kΩ -> 10k
- R11: renamed from R9; value 1kΩ -> 1k
- R12: renamed from R16; value 4k7Ω -> 4k7
- R13: renamed from R10; value 4k7Ω -> 4k7
- R14: renamed from R1; value 2k2Ω -> 2k2
- R15: renamed from R17; value 1kΩ -> 1k
- R16: renamed from R11; value 1kΩ -> 1k
- R17: renamed from R18; value 4k7Ω -> 4k7
- R18: renamed from R12; value 4k7Ω -> 4k7
- R19: value 1kΩ -> 1k
- R2: renamed from R6; value 4k7Ω -> 4k7
- R20: renamed from R21; value 1kΩ -> 1k
- R21: renamed from R20; value 4k7Ω -> 4k7
- R22: value 4k7Ω -> 4k7
- R3: renamed from R13; value 1kΩ -> 1k
- R4: renamed from R7; value 1kΩ -> 1k
- R5: renamed from R14; value 4k7Ω -> 4k7
- R6: renamed from R8; value 4k7Ω -> 4k7
- R7: renamed from R15; value 1kΩ -> 1k
- R8: renamed from R2; value 10kΩ -> 10k
- R9: renamed from R3; value 10kΩ -> 10k
- RN1, RN2: value 100kΩ -> 100k
- RN3: value 10kΩ -> 10k
- U3: value (none) -> 0.96 Inch OLED I2C Display Module
- renumbered C1 to C2, D2 to D1, D6 to D2, D7 to D4, D4 to D5, D1 to D6, D8 to D7, D5 to D8, J2 to J1, J1 to J11, J6 to J2, J7 to J4, J4 to J5, J8 to J6, J5 to J7, J9 to J8, J10 to J9, U4 to U2, U5 to U4, U2 to U6
Connections:
- net +5V: now also C5.1, C6.1, C7.1, D11.1 (K), U5.14 (VCC); no longer R10.1, R9.1
- net CLOCK IN: now also U5.4
- net GND: now also C5.2, C6.2, C7.2, D12.2 (A), J10.S (SHEILD), R24.2, U5.11, U5.13, U5.5, U5.7 (GND), U5.9
- net at RN1.2 (R1): now also U1.7 (QH), U2.9 (A7)
- net at RN1.3 (R2): now also U1.6 (QG), U2.8 (A6)
- net at RN1.4 (R3): now also U1.5 (QF), U2.7 (A5)
- net at RN1.5 (R4): now also U1.4 (QE), U2.6 (A4)
- net at RN1.6 (R5): now also U1.3 (QD), U2.5 (A3)
- net at RN1.7 (R6): now also U1.2 (QC), U2.4 (A2)
- net at RN1.8 (R7): now also U1.1 (QB), U2.3 (A1)
- net at RN1.9 (R8): now also U1.15 (QA), U2.2 (A0)
- net at JP1.2 (C), U3.2 (VCC): now also R10.1, R9.1
- new net: J10.T (SIG), R23.1, R24.1
- new net: D11.2 (A), D12.1 (K), R23.2, U5.1
- new net: U5.2, U5.3
- no-connect marks 32 -> 37
Other:
- note added: "EXTERNAL CLOCK IN CONDITIONING"
- note added: "GATE BUFFERS"
- note added: "GATE SHIFT OUT"
- note added: "MISC BUFFERS"
- note added: "SWITCH SHIFT IN"
- moved on the sheet: A1, C1, C2, C3, C4, D1, D10, D2, D3, D4, D5, D6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

Commit message: revsion A of pcb first iteration
Parts:
- added H1, H2, H3, H4: MountingHole_Pad, MountingHole:MountingHole_2.2mm_M2_Pad_TopBottom, symbol Mechanical:MountingHole_Pad
- SW2: value MUTE 1 -> MUTE1; symbol Switch:SW_SPST -> IMNOTWOPR:SW_SPST
- SW3: value MUTE 2 -> MUTE2; symbol Switch:SW_SPST -> IMNOTWOPR:SW_SPST
- SW4: value MUTE 3 -> MUTE3; symbol Switch:SW_SPST -> IMNOTWOPR:SW_SPST
- SW5: value MUTE 4 -> MUTE4; symbol Switch:SW_SPST -> IMNOTWOPR:SW_SPST
- SW6: value MUTE 5 -> MUTE5; symbol Switch:SW_SPST -> IMNOTWOPR:SW_SPST
- SW7: value MUTE 6 -> MUTE6; symbol Switch:SW_SPST -> IMNOTWOPR:SW_SPST
- SW8: value MUTE 7 -> MUTE7; symbol Switch:SW_SPST -> IMNOTWOPR:SW_SPST
- SW9: value MUTE 8 -> MUTE8; symbol Switch:SW_SPST -> IMNOTWOPR:SW_SPST
Connections:
- net GND: now also SW2.3 (C), SW3.3 (C), SW4.3 (C), SW5.3 (C), SW6.3 (C), SW7.3 (C), SW8.3 (C), SW9.3 (C), H1.1, H2.1, H3.1, H4.1; no longer SW2.2 (B), SW3.2 (B), SW4.2 (B), SW5.2 (B), SW6.2 (B), SW7.2 (B), SW8.2 (B), SW9.2 (B)
- net at RN3.7 (R6), U6.4 (D5): now also SW6.1, SW7.2 (B); no longer SW7.1 (A)
- net at RN3.3 (R2), U6.12 (D1): now also SW2.1, SW3.2 (B); no longer SW3.1 (A)
- net at RN3.6 (R5), U6.3 (D4): now also SW5.1, SW6.2 (B); no longer SW6.1 (A)
- net at RN3.8 (R7), U6.5 (D6): now also SW7.1, SW8.2 (B); no longer SW8.1 (A)
- net at RN3.2 (R1), U6.11 (D0): now also SW2.2 (B); no longer SW2.1 (A)
- net at RN3.4 (R3), U6.13 (D2): now also SW3.1, SW4.2 (B); no longer SW4.1 (A)
- net at RN3.5 (R4), U6.14 (D3): now also SW4.1, SW5.2 (B); no longer SW5.1 (A)
- net at RN3.9 (R8), U6.6 (D7): now also SW8.1, SW9.2 (B); no longer SW9.1 (A)
- net at J11.15 (-12V): no longer J11.16 (P16)
- net at J11.7 (12V): no longer J11.8 (+12V)
- no-connect marks 37 -> 41
