File: hardware/Gateometry.kicad_pcb (KiCad board)
At the start: 2 copper layers, 105.1 x 100 mm, 66 parts, among them J1 POWER, J10 CLOCK OUT, J2 GATE1, J3 GATE3, J4 GATE5, J5 GATE7, J6 GATE2, J7 GATE4, J8 GATE6, J9 GATE8, SW1 RUN/STOP, SW2 MUTE 1, SW3 MUTE 2, SW4 MUTE 3, SW5 MUTE 4, SW6 MUTE 5, SW7 MUTE 6, SW8 MUTE 7, SW9 MUTE 8, U1 74HC595, U2 74HC165, U4 74HCT541, U5 74HCT541

Commit message: initial final rev A schematic
Parts:
- moved R4 113.6 mm to (256.5, 116.5)
- moved C2 113.6 mm to (254.6, 122.2)
- moved R3 113.6 mm to (253.3, 114.0)
- moved A1 102.9 mm to (241.9, 84.8)
- moved RN3 78.8 mm to (233.7, 159.1)
- moved J1 76.7 mm to (236.8, 145.1)
- moved RN2 76.7 mm to (236.8, 137.8)
- moved U2 76.7 mm to (213.3, 117.8)
- moved U4 76.7 mm to (236.8, 125.4)
- moved U5 76.7 mm to (217.8, 126.7)
- moved D1 57.2 mm to (217.9, 75.9)
- moved ENC1 57.2 mm to (217.9, 61.9)
- moved U1 57.2 mm to (217.9, 98.1)
- moved C1 57.2 mm to (223.6, 94.9)
- moved C3 57.2 mm to (212.2, 90.5)
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Other:
- outline, holes or cut-outs redrawn

Commit message: revsion A of pcb first iteration
Parts:
- added C5: 100n, Capacitor_THT:C_Disc_D3.0mm_W1.6mm_P2.50mm, B.Cu at (133.9, 77.8)
- added C6: 100n, Capacitor_THT:C_Disc_D3.0mm_W1.6mm_P2.50mm, B.Cu at (146.6, 82.9)
- added C7: 100n, Capacitor_THT:C_Disc_D3.0mm_W1.6mm_P2.50mm, B.Cu at (140.2, 128.6)
- added D11: BAT85, Diode_THT:D_DO-35_SOD27_P7.62mm_Horizontal, B.Cu at (136.4, 131.1)
- added D12: BAT85, Diode_THT:D_DO-35_SOD27_P7.62mm_Horizontal, B.Cu at (128.8, 133.7)
- added H1: MountingHole_Pad, MountingHole:MountingHole_2.2mm_M2_Pad_TopBottom, F.Cu at (94.7, 53.0)
- added H2: MountingHole_Pad, MountingHole:MountingHole_2.2mm_M2_Pad_TopBottom, F.Cu at (188.3, 53.0)
- added H3: MountingHole_Pad, MountingHole:MountingHole_2.2mm_M2_Pad_TopBottom, F.Cu at (94.7, 147.0)
- added H4: MountingHole_Pad, MountingHole:MountingHole_2.2mm_M2_Pad_TopBottom, F.Cu at (188.3, 147.0)
- added J10: CLOCK IN, Desval27:Jack_3.5mm_QingPu_WQP-PJ398SM_Vertical, F.Cu at (123.1, 140.6)
- added R23: 22k, Resistor_THT:R_Axial_DIN0207_L6.3mm_D2.5mm_P2.54mm_Vertical, B.Cu at (126.3, 136.2)
- added R24: 100k, Resistor_THT:R_Axial_DIN0207_L6.3mm_D2.5mm_P2.54mm_Vertical, B.Cu at (120.5, 136.2)
- added U5: 74HCT14, Package_DIP:DIP-14_W7.62mm_LongPads, B.Cu at (136.4, 137.5)
- C1: renamed from C2; value 10µF -> 47µ
- R1: renamed from R5; value 1kΩ -> 1k
- R10: renamed from R4; value 10kΩ -> 10k
- R11: renamed from R9; value 1kΩ -> 1k
- R12: renamed from R16; value 4k7Ω -> 4k7
- R13: renamed from R10; value 4k7Ω -> 4k7
- R14: renamed from R1; value 2k2Ω -> 2k2
- R15: renamed from R17; value 1kΩ -> 1k
- R16: renamed from R11; value 1kΩ -> 1k
- R17: renamed from R18; value 4k7Ω -> 4k7
- R18: renamed from R12; value 4k7Ω -> 4k7
- R19: value 1kΩ -> 1k
- R2: renamed from R6; value 4k7Ω -> 4k7
- R20: renamed from R21; value 1kΩ -> 1k
- R21: renamed from R20; value 4k7Ω -> 4k7
- R22: value 4k7Ω -> 4k7
- R3: renamed from R13; value 1kΩ -> 1k
- R4: renamed from R7; value 1kΩ -> 1k
- R5: renamed from R14; value 4k7Ω -> 4k7
- R6: renamed from R8; value 4k7Ω -> 4k7
- R7: renamed from R15; value 1kΩ -> 1k
- R8: renamed from R2; value 10kΩ -> 10k
- R9: renamed from R3; value 10kΩ -> 10k
- RN1, RN2: value 100kΩ -> 100k; moved to B.Cu
- RN3: value 10kΩ -> 10k
- SW2: value MUTE 1 -> MUTE1
- SW3: value MUTE 2 -> MUTE2
- SW4: value MUTE 3 -> MUTE3
- SW5: value MUTE 4 -> MUTE4
- SW6: value MUTE 5 -> MUTE5
- SW7: value MUTE 6 -> MUTE6
- SW8: value MUTE 7 -> MUTE7
- SW9: value MUTE 8 -> MUTE8
- U2: renamed from U4; moved to B.Cu
- U3: value ~ -> 0.96 Inch OLED I2C Display Module
- U4: renamed from U5; moved to B.Cu
- moved R1 144.7 mm to (102.8, 54.3)
- moved R4 142.3 mm to (102.8, 74.6)
- moved R11 140.8 mm to (102.8, 94.9)
- moved R16 140.4 mm to (102.8, 115.2)
- moved R2 139.0 mm to (109.8, 54.3), turned to 0 degrees
- moved R3 137.4 mm to (102.8, 64.4)
- moved R6 136.1 mm to (109.8, 74.6), turned to 0 degrees
- moved R7 135.3 mm to (102.8, 84.8)
- moved R15 134.4 mm to (102.8, 105.1)
- moved R13 134.2 mm to (109.8, 94.9), turned to 0 degrees
- moved R20 133.7 mm to (102.8, 135.6)
- moved R19 133.1 mm to (102.8, 125.4)
- moved R5 131.5 mm to (109.8, 64.4), turned to 0 degrees
- moved J11 130.2 mm to (132.6, 67.0)
- moved R18 129.9 mm to (109.8, 115.2), turned to 0 degrees
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- renumbered C1 to C2, D2 to D1, D6 to D2, D7 to D4, D4 to D5, D1 to D6, D8 to D7, D5 to D8, J2 to J1, J1 to J11, J6 to J2, J7 to J4, J4 to J5, J8 to J6, J5 to J7, J9 to J8, J10 to J9, U2 to U6
Connections:
- J11 pad 15: Net-(J1-P16) -> unconnected-(J11--12V-Pad15)
- J11 pad 16: Net-(J1-P16) -> unconnected-(J11-P16-Pad16)
- J11 pad 7: Net-(J1-12V) -> unconnected-(J11-12V-Pad7)
- J11 pad 8: Net-(J1-12V) -> unconnected-(J11-+12V-Pad8)
- R10 pad 1: +5V -> Net-(JP1-C)
- R9 pad 1: +5V -> Net-(JP1-C)
- RN1 pad 2: unconnected-(RN1-R1-Pad2) -> Net-(RN1-R1)
- RN1 pad 3: unconnected-(RN1-R2-Pad3) -> Net-(RN1-R2)
- RN1 pad 4: unconnected-(RN1-R3-Pad4) -> Net-(RN1-R3)
- RN1 pad 5: unconnected-(RN1-R4-Pad5) -> Net-(RN1-R4)
- RN1 pad 6: unconnected-(RN1-R5-Pad6) -> Net-(RN1-R5)
- RN1 pad 7: unconnected-(RN1-R6-Pad7) -> Net-(RN1-R6)
- RN1 pad 8: unconnected-(RN1-R7-Pad8) -> Net-(RN1-R7)
- RN1 pad 9: unconnected-(RN1-R8-Pad9) -> Net-(RN1-R8)
- SW2 pad 1: Net-(RN3-R1) -> unconnected-(SW2-Pad1)
- SW2 pad 2: GND -> Net-(RN3-R1)
- SW2 pad 3: (no net) -> GND
- SW3 pad 1: Net-(RN3-R2) -> unconnected-(SW3-Pad1)
- SW3 pad 2: GND -> Net-(RN3-R2)
- SW3 pad 3: (no net) -> GND
- SW4 pad 1: Net-(RN3-R3) -> unconnected-(SW4-Pad1)
- SW4 pad 2: GND -> Net-(RN3-R3)
- SW4 pad 3: (no net) -> GND
- SW5 pad 1: Net-(RN3-R4) -> unconnected-(SW5-Pad1)
- SW5 pad 2: GND -> Net-(RN3-R4)
- SW5 pad 3: (no net) -> GND
- SW6 pad 1: Net-(RN3-R5) -> unconnected-(SW6-Pad1)
- SW6 pad 2: GND -> Net-(RN3-R5)
- SW6 pad 3: (no net) -> GND
- SW7 pad 1: Net-(RN3-R6) -> unconnected-(SW7-Pad1)
- SW7 pad 2: GND -> Net-(RN3-R6)
- SW7 pad 3: (no net) -> GND
- SW8 pad 1: Net-(RN3-R7) -> unconnected-(SW8-Pad1)
- SW8 pad 2: GND -> Net-(RN3-R7)
- SW8 pad 3: (no net) -> GND
- SW9 pad 1: Net-(RN3-R8) -> unconnected-(SW9-Pad1)
- SW9 pad 2: GND -> Net-(RN3-R8)
- SW9 pad 3: (no net) -> GND
- U1 pad 1: Net-(U1-QB) -> Net-(RN1-R7)
- U1 pad 15: Net-(U1-QA) -> Net-(RN1-R8)
- U1 pad 2: Net-(U1-QC) -> Net-(RN1-R6)
- U1 pad 3: Net-(U1-QD) -> Net-(RN1-R5)
- U1 pad 4: Net-(U1-QE) -> Net-(RN1-R4)
- U1 pad 5: Net-(U1-QF) -> Net-(RN1-R3)
- U1 pad 6: Net-(U1-QG) -> Net-(RN1-R2)
- U1 pad 7: Net-(U1-QH) -> Net-(RN1-R1)
- U2 pad 2: Net-(U1-QA) -> Net-(RN1-R8)
- U2 pad 3: Net-(U1-QB) -> Net-(RN1-R7)
- U2 pad 4: Net-(U1-QC) -> Net-(RN1-R6)
- U2 pad 5: Net-(U1-QD) -> Net-(RN1-R5)
- U2 pad 6: Net-(U1-QE) -> Net-(RN1-R4)
- U2 pad 7: Net-(U1-QF) -> Net-(RN1-R3)
- U2 pad 8: Net-(U1-QG) -> Net-(RN1-R2)
- U2 pad 9: Net-(U1-QH) -> Net-(RN1-R1)
Routing:
- net GND: track 0.00 -> 619.1 mm, vias 0 -> 2
- net +5V: track 0.00 -> 282.5 mm, vias 0 -> 1
- net Net-(A1-A5): track 0.00 -> 107.0 mm, vias 0 -> 1
- net Net-(A1-A4): track 0.00 -> 102.6 mm, vias 0 -> 1
- net +3V3: track 0.00 -> 77.7 mm, vias 0 -> 1
- net Net-(A1-D2): track 0.00 -> 69.5 mm, vias 0 -> 1
- net Net-(RN3-R1): track 0.00 -> 65.6 mm
- net Net-(A1-D3): track 0.00 -> 58.0 mm, vias 0 -> 1
- net Net-(RN3-R2): track 0.00 -> 57.4 mm
- net Net-(A1-A0): track 0.00 -> 57.0 mm, vias 0 -> 1
- net Net-(U4-Y0): track 0.00 -> 56.2 mm
- net Net-(U2-Y0): track 0.00 -> 53.3 mm
- net Net-(A1-A1): track 0.00 -> 50.7 mm, vias 0 -> 2
- net Net-(RN3-R3): track 0.00 -> 49.8 mm
- net Net-(U2-Y1): track 0.00 -> 44.9 mm
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- added copper zone on B.Cu, net +5V
- added copper zone on F.Cu, net +5V
- added copper zone on B.Cu, net GND
- added copper zone on F.Cu, net GND
Other:
- board size 105.1 x 100 mm -> 99.6 x 100 mm
- board text added: "${COMPANY} | ${TITLE} | ${COMMENT2} | REV ${REVISION} | ${CURRENT_DATE} ${COMMENT1}"
- board text added: "+3V3"
- board text added: "+5V"

Commit message: panel work
Parts:
- moved SW1 0.34 mm to (170.4, 84.8)
