File: panel/GateometryPanel.kicad_pcb (KiCad board)
At the start: 2 copper layers, 101.2 x 128.4 mm, 38 parts

Commit message: first revision A of board and panel
Parts:
- added REF**: BTN_6mm_Tact_Cover, Desval27_Panel:BTN_6mm_Tact_Cover, F.Cu at (125.5, 83.3)
- moved <Designator>? 0.17 mm to (97.5, 52.1)
Other:
- board text added: "${COMPANY} - ${TITLE} - ${COMMENT2} - REV ${REVISION} - ${CURRENT_DATE} ${COMMENT1}"
- board text added: "GATE"
- board text added: "IN"
- board text added: "MENU/OK"
- board text added: "MUTE"
- board text added: "START/STOP"
- board text removed: "EXT IN"
- board text removed: "MENU"
- board text removed: "RUN/STOP"
